File: USB_SPDTK2/Controller.kicad_sch (KiCad schematic)
At the start: 42 parts, among them J1 USB_B_Micro, J2 TagConnectTC2050, J3 Conn_02x08_Odd_Even, SW1 SW_Push, SW2 SW_Push, U3 STM32F411RETx, U4 93LC66AT-IOT, U6 L293DD, Y1 16M 20pF 3225

Commit message: Update to v1.1, fix incorrect footprint for L293DD
Parts:
- removed U6: L293DD, Package_SO:SO-20_12.8x7.5mm_P1.27mm, symbol Driver_Motor:L293D
- added U3: L293DD, Package_SO:SO-20_12.8x7.5mm_P1.27mm, symbol mf_lib:L293DD
- renumbered C15 to C14, C21 to C16, C20 to C21, R18 to R12, R17 to R18
Connections:
- net +VSW: now also U3.10 (VCC2)
- net GND: now also U3.14 (GND), U3.15 (GND), U3.16 (GND), U3.17 (GND), U3.4 (GND), U3.5 (GND), U3.6 (GND), U3.7 (GND)
- net S1D: now also U3.9 (2A)
- net S1D_OUT: now also U3.8 (2Y)
- net S1U: now also U3.2 (1A)
- net S1U_OUT: now also U3.3 (1Y)
- net S2D: now also U3.19 (4A)
- net S2D_OUT: now also U3.18 (4Y)
- net S2U: now also U3.12 (3A)
- net S2U_OUT: now also U3.13 (3Y)
- net SW_Enable: now also U3.1 (EN1,2), U3.11 (EN3,4)
- net VBUS: now also U3.20 (VCC1)

Commit message: Submitted to JLCPCB.  Needed an in-stock part for D7
Parts:
- D4: LCSC C434423 -> C125094
Changed lines of the file:
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@@
 			)
 		)
-		(property "LCSC" "C434423"
+		(property "LCSC" "C125094"
 			(at 187.96 106.68 0)
 			(effects
